File: cad/mainboard/untitled.sch (EAGLE design)
At the start: 6 parts

Commit message: cad
Parts:
- added M1, M2, M3, M4: (no value), pinhead:PINHD-1X6
- added X1, X2: (no value), con-wago-500:W237-102
Connections:
- new net M1+: M1.1
- new net M1-: M1.2
- new net M1S1: M1.5
- new net M1S2: M1.6
- new net M2+: M2.1
- new net M2-: M2.2
- new net M2S1: M2.5
- new net M2S2: M2.6
- new net M3+: M3.1
- new net M3-: M3.2
- new net M3S1: M3.5
- new net M3S2: M3.6
- new net M4+: M4.1
- new net M4-: M4.2
- new net M4S1: M4.5
- new net M4S2: M4.6
- net +12V: now also X1-1.KL
- net +5V: now also M1.4, M2.4, M3.4, M4.4, X2-1.KL
- net GND: now also M1.3, M2.3, M3.3, M4.3, X1-2.KL, X2-2.KL

Commit message: board
Parts:
- removed BME280: (no value), pinhead:PINHD-1X6
- added 1K, 1K1, 1K3, 1K4, 1K5, 1K6, R3: 1k, rcl:R-EU_0207/10
- added 1K2: 1.8k, rcl:R-EU_0207/10
- added BACK, FRONT1, FRONT2, MISC: (no value), pinhead:PINHD-1X5
- added C2, C3, C4: (no value), Adafruit DRV8871:MICROBUILDER_CAP_ELECTROLYTICPTH_3.5MMGRID_10MMDIA
- added I2C1, I2C2, I2C3, IN, TRIG: (no value), pinhead:PINHD-1X4
- added M1DRV1, M1DRV2, M1DRV3: (no value), Adafruit DRV8871:MICROBUILDER_DRV8871
- added R1, R4, R5: 30k, rcl:R-EU_0207/10
- added T1, T2, T3, T4: 2N3904, transistor:2N3904
- added UART: (no value), con-wago-500:W237-102
- R2: value (none) -> 30k
- renumbered U1 to M1DRV
Connections:
- removed net M1S1: M1.5
- removed net M1S2: M1.6
- removed net M2S1: M2.5
- removed net M2S2: M2.6
- removed net M3S1: M3.5
- removed net M3S2: M3.6
- removed net M4S1: M4.5
- removed net M4S2: M4.6
- new net +3V3: 1K.1, 3.3V.1, I2C1.4, I2C2.4, I2C3.4, R3.1
- new net ARM2: BACK.1, GND.17
- new net IN: IN.1, T4.C
- new net N$1: M1DRV1.ILIM, R1.1
- new net N$10: 1K3.2, TRIG.3
- new net N$11: IN.3, T2.C
- new net N$12: 1K4.1, T2.B
- new net N$13: 1K4.2, TRIG.2
- new net N$14: IN.4, T3.C
- new net N$15: 1K5.1, T3.B
- new net N$16: 1K5.2, TRIG.1
- new net N$18: 1K6.1, T4.B
- new net N$19: 1K6.2, TRIG.4
- new net N$2: M1DRV2.ILIM, R4.1
- new net N$3: 1K1.1, GND.9
- new net N$4: M1DRV3.ILIM, R5.1
- new net N$5: GND.11, UART-2.KL
- new net N$6: GND.12, UART-1.KL
- new net N$7: IN.2, T1.C
- new net N$8: 1K3.1, T1.B
- new net P0: GND.14, MISC.1
- new net P10: 3.3V.16, M2.6
- new net P11: 3.3V.17, M3.5
- new net P12: 3.3V.18, M3.6
- new net P13: 3.3V.19, M4.5
- new net P14: 3.3V.20, M4.6
- new net P15LASERX: 3.3V.8, FRONT2.4
- new net P16LASERY: 3.3V.9, FRONT2.3
- new net P17LASERTRIG: 3.3V.10, FRONT2.2
- new net P18SDA: 1K.2, 3.3V.11, I2C1.1, I2C2.1, I2C3.1
- new net P19SCL: GND.20, I2C1.2, I2C2.2, I2C3.2, R3.2
- new net P1ARM3: BACK.5, GND.4
- new net P20: GND.19, MISC.3
- new net P21: GND.18, MISC.2
- new net P2ARM4: BACK.4, GND.5
- new net P3: 3.3V.13, M1.6
- new net P35SONAR: FRONT1.3, GND.13
- new net P38SONARTRIG: FRONT1.5, GND.10
- new net P39SONARECHO: 1K1.2, 1K2.2, FRONT1.4
- new net P4: 3.3V.4, MISC.5
- new net P40: M1DRV.IN1, M1DRV1.IN1, M1DRV2.IN1, M1DRV3.IN1
- new net P40PWM2: GND.8
- new net P41PWM1: GND.7, M1DRV.IN2, M1DRV1.IN2, M1DRV2.IN2, M1DRV3.IN2
- new net P42ARM1: BACK.3, GND.6
- new net P43: GND.2
- new net P44: GND.3
- new net P45REARBUMP: BACK.2, GND.15
- new net P46FRONTBUMP: 3.3V.14, FRONT2.1
- new net P48LED: FRONT1.2, GND.16
- new net P5BUZZER: 3.3V.5, FRONT1.1
- new net P6: 3.3V.6, MISC.4
- new net P7STEER: 3.3V.7, FRONT2.5
- new net P8: 3.3V.12, M1.5
- new net P9: 3.3V.15, M2.5
- net +12V: now also C2.+, C3.+, C4.+, M1DRV1.VM, M1DRV2.VM, M1DRV3.VM
- net +5V: now also 3.3V.21; no longer BME280.6
- net GND: now also 1K2.1, 3.3V.22, C2.-, C3.-, C4.-, GND.21, GND.22, I2C1.3, I2C2.3, I2C3.3, M1DRV1.GND, M1DRV1.PGND, M1DRV2.GND, M1DRV2.PGND, M1DRV3.GND, M1DRV3.PGND, R1.2, R4.2, R5.2, T1.E, T2.E, T3.E, T4.E; no longer BME280.5
- net M1+: now also M1DRV.OUT1
- net M1-: now also M1DRV.OUT2
- net M2+: now also M1DRV1.OUT1
- net M2-: now also M1DRV1.OUT2
- net M3+: now also M1DRV2.OUT1
- net M3-: now also M1DRV2.OUT2
- net M4+: now also M1DRV3.OUT1
- net M4-: now also M1DRV3.OUT2
Other:
- moved on the sheet: 3.3V, C1, GND, M1, M2, M3, M4, X1-1, X1-2, X2-1, X2-2

Commit message: pcb
Connections:
- removed net P40: M1DRV.IN1, M1DRV1.IN1, M1DRV2.IN1, M1DRV3.IN1
- net P40PWM2: now also M1DRV.IN1, M1DRV1.IN1, M1DRV2.IN1, M1DRV3.IN1
Changed lines of the file:
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@@
 <setting verticaltext="up"/>
 </settings>
-<grid distance="0.1" unitdist="inch" unit="inch" style="lines" multiple="1" display="yes" altdistance="0.01" altunitdist="inch" altunit="inch"/>
+<grid distance="0.1" unitdist="inch" unit="inch" style="lines" multiple="1" display="no" altdistance="0.01" altunitdist="inch" altunit="inch"/>
 <layers>
 <layer number="1" name="Top" color="4" fill="1" visible="no" active="no"/>
@@
 </segment>
 </net>
-<net name="P40" class="0">
-<segment>
-<wire x1="-68.58" y1="-27.94" x2="-66.04" y2="-27.94" width="0.1524" layer="91" grouprefs="DRIVER4"/>
-<label x="-66.04" y="-27.94" size="1.778" layer="95" xref="yes" grouprefs="DRIVER4"/>
-<pinref part="M1DRV3" gate="G$1" pin="IN1"/>
-</segment>
-<segment>
-<wire x1="-68.58" y1="27.94" x2="-66.04" y2="27.94" width="0.1524" layer="91" grouprefs="DRIVER3"/>
-<label x="-66.04" y="27.94" size="1.778" layer="95" xref="yes" grouprefs="DRIVER3"/>
-<pinref part="M1DRV2" gate="G$1" pin="IN1"/>
-</segment>
-<segment>
-<wire x1="-68.58" y1="83.82" x2="-66.04" y2="83.82" width="0.1524" layer="91" grouprefs="DRIVER2"/>
-<label x="-66.04" y="83.82" size="1.778" layer="95" xref="yes" grouprefs="DRIVER2"/>
-<pinref part="M1DRV1" gate="G$1" pin="IN1"/>
-</segment>
-<segment>
-<pinref part="M1DRV" gate="G$1" pin="IN1"/>
-<wire x1="-68.58" y1="139.7" x2="-66.04" y2="139.7" width="0.1524" layer="91" grouprefs="DRIVER1"/>
-<label x="-66.04" y="139.7" size="1.778" layer="95" xref="yes" grouprefs="DRIVER1"/>
-</segment>
-</net>
 <net name="P39SONARECHO" class="0">
 <segment>
@@
 <label x="106.68" y="73.66" size="1.778" layer="95" rot="R180" xref="yes"/>
 </segment>
-</net>
+<segment>
+<wire x1="-68.58" y1="-27.94" x2="-66.04" y2="-27.94" width="0.1524" layer="91" grouprefs="DRIVER4"/>
+<label x="-66.04" y="-27.94" size="1.778" layer="95" xref="yes" grouprefs="DRIVER4"/>
+<pinref part="M1DRV3" gate="G$1" pin="IN1"/>
+</segment>
+<segment>
+<wire x1="-68.58" y1="27.94" x2="-66.04" y2="27.94" width="0.1524" layer="91" grouprefs="DRIVER3"/>
+<label x="-66.04" y="27.94" size="1.778" layer="95" xref="yes" grouprefs="DRIVER3"/>
+<pinref part="M1DRV2" gate="G$1" pin="IN1"/>
+</segment>
+<segment>
+<wire x1="-68.58" y1="83.82" x2="-66.04" y2="83.82" width="0.1524" layer="91" grouprefs="DRIVER2"/>
+<label x="-66.04" y="83.82" size="1.778" layer="95" xref="yes" grouprefs="DRIVER2"/>
+<pinref part="M1DRV1" gate="G$1" pin="IN1"/>
+</segment>
+<segment>
+<pinref part="M1DRV" gate="G$1" pin="IN1"/>
+<wire x1="-68.58" y1="139.7" x2="-66.04" y2="139.7" width="0.1524" layer="91" grouprefs="DRIVER1"/>
+<label x="-66.04" y="139.7" size="1.778" layer="95" xref="yes" grouprefs="DRIVER1"/>
+</segment>
+</net>
